File: Robot/ESP PCB/ESP PCB.kicad_sch (KiCad schematic)
At the start: 1 part, among them U1 ESP32-S3-DevKitC

Commit message: cad
Parts:
- added J1: Conn_01x15_Socket, symbol Connector:display_driver_symbol
Changed lines of the file:
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@@
     (pin "9")
     (instances
-      (project ""
+      (project "ESP PCB"
         (path "/d2d679ee-cdfd-4a56-9660-534e55f0cb8f"
           (reference "U1") (unit 1)
         )
       )
+    )
+  )
+  (symbol (lib_id "Connector:display_driver_symbol") (at 180.34 58.42 0) (unit 1)
+    (in_bom yes) (on_board yes) (dnp no) (fields_autoplaced)
+    (property "Reference" "J1" (at 181.61 57.785 0)
+      (effects (font (size 1.27 1.27)) (justify left))
+    )
+    (property "Value" "Conn_01x15_Socket" (at 181.61 60.325 0)
+      (effects (font (size 1.27 1.27)) (justify left))
+    )
+    (property "Footprint" "" (at 180.34 58.42 0)
+      (effects (font (size 1.27 1.27)) hide)
+    )
+    (property "Datasheet" "~" (at 180.34 58.42 0)
+      (effects (font (size 1.27 1.27)) hide)
+    )
+    (pin "1")
+    (pin "10")
+    (pin "11")
+    (pin "12")
+    (pin "13")
+    (pin "14")
+    (pin "15")
+    (pin "2")
+    (pin "3")
+    (pin "4")
+    (pin "5")
+    (pin "6")
+    (pin "7")
+    (pin "8")
+    (pin "9")
+    (instances
+      (project "ESP PCB"
+        (path "/d2d679ee-cdfd-4a56-9660-534e55f0cb8f"
+          (reference "J1") (unit 1)
+        )
+      )
