File: dsi_esp32/dsi_esp.kicad_sch (KiCad schematic)
At the start: 14 parts, among them U1 ndsPADS, U2 ESP32-S3-WROOM-1

Commit message: working prototype that sends the images automatically over esp-now and is able to display. esp-now is too slow however so we need to switch from it
Parts:
- removed POWER1, PROGRAM1: ~, Ilya_Teach:1X2_SMALL_TH, symbol Ilya_Teach:CONN_DEBUGA
- added J1: ~, SparkFun-Connectors:1X04, symbol SparkFun-Connectors:CONN_04PTH
Connections:
- net GND: now also J1.2; no longer R3.2
- net RXD: now also J1.3
- net SPI_MISO: now also U1.15 (D6)
- net TXD: now also J1.4
- net VCC: now also J1.1
- net WIFI_IND: now reaches U2.16 (GPIO46)
- net WIFI_IND: now also R3.2
