File: Robot/flexible PCB layered coil/flex_pcb_coil/flex_pcb_coil.kicad_sch (KiCad schematic)
At the start: 1 part

Commit message: dsdasdkan
Parts:
- removed D1: LED_Pad, symbol Device:LED_Pad
- added J1, J2: Conn_01x01_Pin, Connector_PinHeader_2.54mm:PinHeader_1x01_P2.54mm_Vertical, symbol Connector:Conn_01x01_Pin
Connections:
- new net: J1.1 (Pin_1), J2.1 (Pin_1)
Changed lines of the file:
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@@
 (kicad_sch (version 20230121) (generator eeschema)
   (paper "A4")
-  (symbol (lib_id "Device:LED_Pad") (at 116.84 96.52 0) (unit 1)
+  (wire (pts (xy 100.33 102.87) (xy 100.33 109.22))
+    (stroke (width 0) (type default))
+  )
+  (symbol (lib_id "Connector:Conn_01x01_Pin") (at 95.25 109.22 0) (unit 1)
     (in_bom yes) (on_board yes) (dnp no) (fields_autoplaced)
-    (property "Reference" "D1" (at 116.84 90.17 0)
+    (property "Reference" "J2" (at 95.885 105.41 0)
       (effects (font (size 1.27 1.27)))
     )
-    (property "Value" "LED_Pad" (at 116.84 92.71 0)
+    (property "Value" "Conn_01x01_Pin" (at 95.885 107.95 0)
       (effects (font (size 1.27 1.27)))
     )
-    (property "Footprint" "" (at 116.84 96.52 0)
+    (property "Footprint" "Connector_PinHeader_2.54mm:PinHeader_1x01_P2.54mm_Vertical" (at 95.25 109.22 0)
       (effects (font (size 1.27 1.27)) hide)
     )
-    (property "Datasheet" "~" (at 116.84 96.52 0)
+    (property "Datasheet" "~" (at 95.25 109.22 0)
       (effects (font (size 1.27 1.27)) hide)
     )
     (pin "1")
-    (pin "2")
-    (pin "3")
     (instances
       (project "flex_pcb_coil"
         (path "/c2967291-a2ef-4fcd-aad3-438aab1728fc"
-          (reference "D1") (unit 1)
+          (reference "J2") (unit 1)
         )
       )
+    )
+  )
+  (symbol (lib_id "Connector:Conn_01x01_Pin") (at 95.25 102.87 0) (unit 1)
+    (in_bom yes) (on_board yes) (dnp no) (fields_autoplaced)
+    (property "Reference" "J1" (at 95.885 99.06 0)
+      (effects (font (size 1.27 1.27)))
+    )
+    (property "Value" "Conn_01x01_Pin" (at 95.885 101.6 0)
+      (effects (font (size 1.27 1.27)))
+    )
+    (property "Footprint" "Connector_PinHeader_2.54mm:PinHeader_1x01_P2.54mm_Vertical" (at 95.25 102.87 0)
+      (effects (font (size 1.27 1.27)) hide)
+    )
+    (property "Datasheet" "~" (at 95.25 102.87 0)
+      (effects (font (size 1.27 1.27)) hide)
+    )
+    (pin "1")
+    (instances
+      (project "flex_pcb_coil"
+        (path "/c2967291-a2ef-4fcd-aad3-438aab1728fc"
+          (reference "J1") (unit 1)
+        )
+      )
